File: design/21_LetsSwamp_Assemble_L/21_LetsSwamp_Assemble_L.sch (KiCad schematic (older format))
At the start: 52 parts, among them J1 MJ-4PP-9, J2 Conn_01x03, SW1 SW_Push, SW10 SW_Push, SW11 SW_Push, SW12 SW_Push, SW13 SW_Push, SW14 SW_Push, SW15 SW_Push, SW16 SW_Push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

Commit message: Modify reference number
Parts:
- renumbered D25 to D49
Changed lines of the file:
@@
 	4725 3850 5475 3850
 $Comp
-L Device:D D25
+L Device:D D49
 U 1 1 63AFB9D2
 P 5825 1625
-F 0 "D25" V 5871 1545 50  0000 R CNN
+F 0 "D49" V 5871 1545 50  0000 R CNN
 F 1 "D" V 5780 1545 50  0000 R CNN
 F 2 "footprints:Diode_TH_SMD" H 5825 1625 50  0001 C CNN
