File: design/21_LetsSwamp_Assemble_L/21_LetsSwamp_Assemble_L.kicad_pcb (KiCad board)
At the start: 2 copper layers, 122.3 x 85 mm, 53 parts, among them J1 MJ-4PP-9, J2 Conn_01x03, SW1 SW_Push, SW10 SW_Push, SW11 SW_Push, SW12 SW_Push, SW13 SW_Push, SW14 SW_Push, SW15 SW_Push, SW16 SW_Push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

Commit message: Hide JLCJLCJLC
Other:
- board text added: "v1.0"
- board text removed: "v0.3"
