File: design/22_LetsSwamp_Assemble_R/22_LetsSwamp_Assemble_R.kicad_pcb (KiCad board)
At the start: 2 copper layers, 122.3 x 85 mm, 52 parts, among them J1 MJ-4PP-9, J2 Conn_01x03, SW26 SW_Push, SW27 SW_Push, SW28 SW_Push, SW29 SW_Push, SW30 SW_Push, SW31 SW_Push, SW32 SW_Push, SW33 SW_Push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

Commit message: Modify reference number
Parts:
- renumbered D26 to D25, D27 to D26, D28 to D27, D29 to D28, D30 to D29, D31 to D30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
