File: design/22_LetsSwamp_Assemble_R/22_LetsSwamp_Assemble_R.kicad_pcb (KiCad board)
At the start: 2 copper layers, 122.3 x 85 mm, 53 parts, among them J1 MJ-4PP-9, J2 Conn_01x03, SW25 SW_Push, SW26 SW_Push, SW27 SW_Push, SW28 SW_Push, SW29 SW_Push, SW30 SW_Push, SW31 SW_Push, SW32 SW_Push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

Commit message: Hide JLCJLCJLC
Other:
- board text added: "v1.0"
- board text removed: "v0.3"
